File: CANShield.kicad_sch (KiCad schematic)
At the start: 92 parts, among them J101 Conn_02x19_Odd_Even, J102 Conn_02x19_Odd_Even, J103 Conn_01x04_Socket, J104 Conn_01x06_Socket, Q101 Si1308EDL, Q102 Si1308EDL, Q103 Si1308EDL, U101 TJA1443ATK/0Z, U102 BD2222G, U103 AT25SF081-XMHD-X, U104 MR20H40

Commit message: pcb in progress
working on pcb layout
Parts:
- added TP114: TestPoint_Small, TestPoint:TestPoint_Pad_D1.0mm, symbol Connector:TestPoint_Small
- renumbered TP116 to TP101, TP101 to TP102, TP102 to TP103, TP103 to TP104, TP104 to TP105, TP117 to TP106, TP105 to TP107, TP118 to TP108, TP106 to TP109, TP107 to TP110, TP108 to TP111, TP115 to TP112, TP114 to TP113, TP109 to TP115, TP111 to TP116, TP113 to TP117, TP110 to TP118, TP112 to TP119
Connections:
- net GND: now also TP114.1
- net CAN0_H renamed CAN0_P
- net CAN0_L renamed CAN0_N
Changed lines of the file:
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@@
 	)
 	(junction
+		(at 273.05 67.31)
+		(diameter 0)
+		(color 0 0 0 0)
+	)
+	(junction
 		(at 307.34 199.39)
 		(diameter 0)
@@
 	(wire
 		(pts
-			(xy 273.05 68.58) (xy 273.05 66.04)
+			(xy 273.05 68.58) (xy 273.05 67.31)
 		)
 		(stroke
@@
 	(wire
 		(pts
+			(xy 273.05 67.31) (xy 273.05 66.04)
+		)
+		(stroke
+			(width 0)
+			(type default)
+		)
+	)
+	(wire
+		(pts
 			(xy 175.26 227.33) (xy 179.07 227.33)
 		)
@@
 		)
 	)
-	(label "CAN0_L"
+	(label "CAN0_N"
 		(at 118.11 229.87 180)
 		(fields_autoplaced yes)
@@
 		)
 	)
-	(label "CAN0_H"
+	(label "CAN0_P"
 		(at 118.11 237.49 180)
 		(fields_autoplaced yes)
@@
 		(on_board yes)
 		(dnp no)
-		(property "Reference" "TP107"
+		(property "Reference" "TP110"
 			(at 123.952 228.346 0)
 			(effects
@@
 			(project "CANShield"
 				(path "/b267ac6b-6338-40f7-a3df-596945dc6f78"
-					(reference "TP107")
+					(reference "TP110")
 					(unit 1)
 				)
@@
 		(on_board yes)
 		(dnp no)
-		(property "Reference" "TP109"
+		(property "Reference" "TP115"
 			(at 282.702 44.196 0)
 			(effects
@@
 			(project "CANShield"
 				(path "/b267ac6b-6338-40f7-a3df-596945dc6f78"
-					(reference "TP109")
+					(reference "TP115")
 					(unit 1)
 				)
@@
 		(on_board yes)
 		(dnp no)
-		(property "Reference" "TP110"
+		(property "Reference" "TP118"
 			(at 285.242 46.736 0)
 			(effects
@@
 			(project "CANShield"
 				(path "/b267ac6b-6338-40f7-a3df-596945dc6f78"
-					(reference "TP110")
+					(reference "TP118")
 					(unit 1)
 				)
@@
 	)
 	(symbol
+		(lib_id "Connector:TestPoint_Small")
+		(at 273.05 67.31 0)
+		(unit 1)
+		(exclude_from_sim no)
+		(in_bom yes)
+		(on_board yes)
+		(dnp no)
+		(property "Reference" "TP114"
+			(at 273.812 67.31 0)
+			(effects
+				(font
+					(size 1.27 1.27)
+				)
+				(justify left)
+			)
+		)
+		(property "Value" "TestPoint_Small"
+			(at 274.32 68.5799 0)
+			(effects
+				(font
+					(size 1.27 1.27)
+				)
+				(justify left)
+				(hide yes)
+			)
+		)
+		(property "Footprint" "TestPoint:TestPoint_Pad_D1.0mm"
+			(at 278.13 67.31 0)
+			(effects
+				(font
+					(size 1.27 1.27)
+				)
+				(hide yes)
+			)
+		)
+		(property "Datasheet" "~"
+			(at 278.13 67.31 0)
+			(effects
+				(font
+					(size 1.27 1.27)
+				)
+				(hide yes)
+			)
+		)
+		(property "Description" "test point"
+			(at 273.05 67.31 0)
+			(effects
+				(font
+					(size 1.27 1.27)
+				)
+				(hide yes)
+			)
+		)
+		(pin "1"
+		)
+		(instances
+			(project "CANShield"
+				(path "/b267ac6b-6338-40f7-a3df-596945dc6f78"
+					(reference "TP114")
+					(unit 1)
+				)
+			)
+		)
+	)
+	(symbol
 		(lib_id "power:+5V")
 		(at 222.25 114.3 0)
@@
 		(on_board yes)
 		(dnp no)
-		(property "Reference" "TP102"
+		(property "Reference" "TP103"
 			(at 51.562 234.696 0)
 			(effects
@@
 			(project "CANShield"
 				(path "/b267ac6b-6338-40f7-a3df-596945dc6f78"
-					(reference "TP102")
+					(reference "TP103")
 					(unit 1)
 				)
@@
 		(on_board yes)
 		(dnp no)
-		(property "Reference" "TP104"
+		(property "Reference" "TP105"
 			(at 51.562 248.666 0)
 			(effects
@@
 			(project "CANShield"
 				(path "/b267ac6b-6338-40f7-a3df-596945dc6f78"
-					(reference "TP104")
+					(reference "TP105")
 					(unit 1)
 				)
@@
 		(on_board yes)
 		(dnp no)
-		(property "Reference" "TP113"
+		(property "Reference" "TP117"
 			(at 282.702 54.356 0)
 			(effects
@@
 			(project "CANShield"
 				(path "/b267ac6b-6338-40f7-a3df-596945dc6f78"
-					(reference "TP113")
+					(reference "TP117")
 					(unit 1)
 				)
@@
 		(on_board yes)
 		(dnp no)
-		(property "Reference" "TP114"
+		(property "Reference" "TP113"
 			(at 264.922 36.576 0)
 			(effects
@@
 			(project "CANShield"
 				(path "/b267ac6b-6338-40f7-a3df-596945dc6f78"
-					(reference "TP114")
+					(reference "TP113")
 					(unit 1)
 				)
@@
 		(on_board yes)
 		(dnp no)
-		(property "Reference" "TP106"
+		(property "Reference" "TP109"
 			(at 112.522 244.856 0)
 			(effects
@@
 			(project "CANShield"
 				(path "/b267ac6b-6338-40f7-a3df-596945dc6f78"
-					(reference "TP106")
+					(reference "TP109")
 					(unit 1)
 				)
@@
 		(on_board yes)
 		(dnp no)
-		(property "Reference" "TP115"
+		(property "Reference" "TP112"
 			(at 240.792 133.096 0)
 			(effects
@@
 			(project "CANShield"
 				(path "/b267ac6b-6338-40f7-a3df-596945dc6f78"
-					(reference "TP115")
+					(reference "TP112")
 					(unit 1)
 				)
@@
 		(on_board yes)
 		(dnp no)
-		(property "Reference" "TP101"
+		(property "Reference" "TP102"
 			(at 51.562 230.886 0)
 			(effects
@@
 			(project "CANShield"
 				(path "/b267ac6b-6338-40f7-a3df-596945dc6f78"
-					(reference "TP101")
+					(reference "TP102")
 					(unit 1)
 				)
@@
 		(on_board yes)
 		(dnp no)
-		(property "Reference" "TP111"
+		(property "Reference" "TP116"
 			(at 282.702 49.276 0)
 			(effects
@@
 			(project "CANShield"
 				(path "/b267ac6b-6338-40f7-a3df-596945dc6f78"
-					(reference "TP111")
+					(reference "TP116")
 					(unit 1)
 				)
@@
 		(on_board yes)
 		(dnp no)
-		(property "Reference" "TP112"
+		(property "Reference" "TP119"
 			(at 285.242 51.816 0)
 			(effects
@@
 			(project "CANShield"
 				(path "/b267ac6b-6338-40f7-a3df-596945dc6f78"
-					(reference "TP112")
+					(reference "TP119")
 					(unit 1)
 				)
@@
 		(on_board yes)
 		(dnp no)
-		(property "Reference" "TP117"
+		(property "Reference" "TP106"
 			(at 54.102 91.186 0)
 			(effects
@@
 			(project "CANShield"
 				(path "/b267ac6b-6338-40f7-a3df-596945dc6f78"
-					(reference "TP117")
+					(reference "TP106")
 					(unit 1)
 				)
@@
 		(on_board yes)
 		(dnp no)
-		(property "Reference" "TP105"
+		(property "Reference" "TP107"
 			(at 55.372 228.346 0)
 			(effects
@@
 			(project "CANShield"
 				(path "/b267ac6b-6338-40f7-a3df-596945dc6f78"
-					(reference "TP105")
+					(reference "TP107")
 					(unit 1)
 				)
@@
 		(on_board yes)
 		(dnp no)
-		(property "Reference" "TP116"
+		(property "Reference" "TP101"
 			(at 51.562 88.646 0)
 			(effects
@@
 			(project "CANShield"
 				(path "/b267ac6b-6338-40f7-a3df-596945dc6f78"
-					(reference "TP116")
+					(reference "TP101")
 					(unit 1)
 				)
@@
 		(on_board yes)
 		(dnp no)
-		(property "Reference" "TP118"
+		(property "Reference" "TP108"
 			(at 56.642 93.726 0)
 			(effects
@@
 			(project "CANShield"
 				(path "/b267ac6b-6338-40f7-a3df-596945dc6f78"
-					(reference "TP118")
+					(reference "TP108")
 					(unit 1)
 				)
@@
 		(on_board yes)
 		(dnp no)
-		(property "Reference" "TP103"
+		(property "Reference" "TP104"
 			(at 51.562 241.046 0)
 			(effects
@@
 			(project "CANShield"
 				(path "/b267ac6b-6338-40f7-a3df-596945dc6f78"
-					(reference "TP103")
+					(reference "TP104")
 					(unit 1)
 				)
@@
 		(on_board yes)
 		(dnp no)
-		(property "Reference" "TP108"
+		(property "Reference" "TP111"
 			(at 123.952 235.966 0)
 			(effects
@@
 			(project "CANShield"
 				(path "/b267ac6b-6338-40f7-a3df-596945dc6f78"
-					(reference "TP108")
+					(reference "TP111")
 					(unit 1)
 				)
