File: CANShield.kicad_pcb (KiCad board)
At the start: 2 copper layers, 70 x 59 mm, 92 parts, among them J101 Conn_02x19_Odd_Even, J102 Conn_02x19_Odd_Even, J103 Conn_01x04_Socket, J104 Conn_01x06_Socket, Q101 Si1308EDL, Q102 Si1308EDL, Q103 Si1308EDL, U101 TJA1443ATK/0Z, U102 BD2222G, U103 AT25SF081-XMHD-X, U104 MR20H40

Commit message: pcb in progress
working on pcb layout
Parts:
- added TP114: TestPoint_Small, TestPoint:TestPoint_Pad_D1.0mm, F.Cu at (162.8, 110.0)
- moved C105 128.1 mm to (110.1, 114.5)
- moved C103 126.9 mm to (110.7, 105.7), turned to 90 degrees
- moved JP104 125.6 mm to (112.2, 112.2), turned to -90 degrees
- moved C101 123.3 mm to (110.4, 103.7)
- moved C108 118.3 mm to (125.0, 116.3), turned to 180 degrees
- moved C102 118.2 mm to (120.2, 109.2), turned to -90 degrees
- moved C104 114.9 mm to (123.7, 113.4), turned to 180 degrees
- moved L102 112.6 mm to (110.1, 115.6)
- moved JP101 111.5 mm to (112.2, 108.6), turned to -90 degrees
- moved L101 110.7 mm to (109.5, 105.7), turned to 90 degrees
- moved C106 110.4 mm to (128.1, 116.3)
- moved R104 109.4 mm to (124.7, 114.9), turned to 180 degrees
- moved R105 109.0 mm to (124.2, 111.2), turned to 90 degrees
- moved TP105 109.0 mm to (114.8, 111.2)
- moved R101 105.1 mm to (119.2, 109.2), turned to -90 degrees
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- renumbered TP116 to TP101, TP101 to TP102, TP102 to TP103, TP103 to TP104, TP104 to TP105, TP117 to TP106, TP105 to TP107, TP118 to TP108, TP106 to TP109, TP107 to TP110, TP108 to TP111, TP115 to TP112, TP114 to TP113, TP109 to TP115, TP111 to TP116, TP113 to TP117, TP110 to TP118, TP112 to TP119
Connections:
- net /CAN0_H renamed /CAN0_P
- net /CAN0_L renamed /CAN0_N
Routing:
- net /SCLK: track 0.00 -> 57.0 mm, vias 0 -> 1
- net /LED0_BLU: track 1.56 -> 55.9 mm, vias 0 -> 1
- net /LED0_GRN: track 1.56 -> 54.6 mm, vias 0 -> 1
- net /LED0_RED: track 1.52 -> 52.8 mm, vias 0 -> 1
- net /CAN0_EN: track 0.00 -> 44.9 mm, vias 0 -> 2
- net /~{CAN0_STB}: track 0.00 -> 39.8 mm, vias 0 -> 1
- net /MOSI: track 0.00 -> 39.1 mm, vias 0 -> 1
- net /CAN0_N: track 0.00 -> 34.4 mm
- net /CAN0_P: track 0.00 -> 32.1 mm
- net /CAN0_RXD: track 0.00 -> 30.8 mm, vias 0 -> 1
- net /~{WP}: track 0.00 -> 30.3 mm, vias 0 -> 1
- net /FLASH_CS: track 0.00 -> 27.4 mm, vias 0 -> 1
- net /CAN0_TXD: track 0.00 -> 26.9 mm, vias 0 -> 1
- net /MISO: track 0.00 -> 26.4 mm, vias 0 -> 1
- net GND: track 4.56 -> 30.3 mm, vias 0 -> 17
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
Commit message: working on PCB
Parts:
- removed TP110, TP111: TestPoint_Small, TestPoint:TestPoint_Pad_D1.0mm
- moved JP103 123.4 mm to (110.0, 97.6)
- moved TP101 121.4 mm to (107.7, 99.7)
- moved TP106 121.4 mm to (107.7, 102.7)
- moved TP108 121.4 mm to (107.7, 105.8)
- moved JP102 119.2 mm to (109.8, 94.0), turned to 180 degrees
- moved D101 118.7 mm to (117.7, 114.7)
- moved TP104 113.7 mm to (109.2, 89.5)
- moved TP102 109.8 mm to (113.0, 89.5)
- moved TP107 108.4 mm to (114.8, 91.7)
- moved TP109 106.2 mm to (117.0, 111.3)
- moved R107 106.0 mm to (117.7, 113.5)
- moved TP103 105.8 mm to (117.0, 89.5)
- moved TP112 86.5 mm to (144.7, 113.3)
- moved R105 2.12 mm to (122.8, 109.7)
- moved C104 1.89 mm to (122.2, 112.3)
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Routing:
- net /CAN0_LED: track 0.00 -> 35.4 mm
- net +5V: track 4.90 -> 31.0 mm, vias 2 -> 4
- net /~{CAN0_STB}: track 39.8 -> 54.7 mm
- net PVCC: track 12.3 -> 25.3 mm
- net Net-(C104-Pad1): track 3.01 -> 13.7 mm, vias 0 -> 2
- net /CAN0_N: track 34.4 -> 24.6 mm
- net /CAN0_P: track 32.1 -> 23.9 mm
- net /PC13: track 0.00 -> 7.16 mm
- net GND: track 30.3 -> 37.2 mm, vias 17 -> 45
- net /PC14: track 0.00 -> 6.73 mm
- net /PC15: track 0.00 -> 6.37 mm
- net +3V3: track 17.5 -> 22.5 mm, vias 7 -> 8
- net Net-(U101-NC): track 8.40 -> 5.70 mm
- net /CAN0_EN: track 44.9 -> 46.9 mm, vias 2 -> 3
- net /~{PRB_FLG}: track 23.2 -> 24.8 mm
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- added copper zone on B.Cu, net GND

Commit message: finished PCB
Parts:
- added G***: LOGO, LOGO, F.Cu at (135.8, 101.6)
- moved TP101 17.8 mm to (122.2, 89.5)
- moved TP106 17.8 mm to (122.2, 92.5)
- moved TP108 17.8 mm to (122.2, 95.6)
- moved TP107 1.60 mm to (116.5, 91.7)
- moved TP103 1.08 mm to (116.5, 88.6)
- moved TP104 0.90 mm to (109.2, 88.6)
- moved TP102 0.80 mm to (113.0, 90.3)
- moved D103 0.08 mm to (131.6, 77.0)
- moved D104 0.08 mm to (138.8, 77.0)
Routing:
- net +5V: track 31.0 -> 76.0 mm
- net /PC13: track 7.16 -> 32.1 mm, vias 0 -> 1
- net /PC14: track 6.73 -> 31.3 mm, vias 0 -> 1
- net GND: track 37.2 -> 60.7 mm, vias 45 -> 57
- net /PC15: track 6.37 -> 29.1 mm, vias 0 -> 1
- net +3V3: track 22.5 -> 27.1 mm
- net /MOSI: track 39.1 -> 35.9 mm
- net /CAN0_RXD: track 30.8 -> 33.3 mm
- net /CAN0_TXD: track 26.9 -> 29.4 mm
- net /PROBE_EN: track 24.7 -> 23.5 mm
- net /USART1_RX: track 22.1 -> 21.0 mm
- net /CAN0_EN: track 46.9 -> 47.9 mm
- net /CAN0_LED: track 35.4 -> 36.4 mm
- added copper zone on In2.Cu, net +3V3
- added copper zone on In1.Cu, net GND
Other:
- copper layers 2 -> 4
- board text added: "+3V3"
- board text added: "+5V"
- board text added: "06/24 PEK"
- board text added: "CAN LED0"
- board text added: "CANShield"
- board text added: "CEN"
- board text added: "CN9"
- board text added: "CRXD"
- board text added: "CTXD"
- board text added: "GND"
- board text added: "MISO"
- board text added: "MOSI"
- board text added: "NXP TJA1443 Testboard"
- board text added: "PC13"
- board text added: "PC14"
- board text added: "PC15"
- board text added: "SCLK"
- board text added: "~{CS}"
- board text added: "~{STB}"
- board text added: "~{WP}"
